Commit message: teleop working on my_robot.urdf

File: urdf/my_robot.urdf (robot description, URDF)
Before this commit: robot my_robot, 7 links, 6 joints
Joints:
- joint base_to_left_wheel: origin xyz=0 -0.23 -0.1 rpy=0 0 1.57 -> xyz=0 0.230 -0.1 rpy=0 0 1.57
- joint base_to_right_wheel: origin xyz=0 0.23 -0.1 rpy=0 0 1.57 -> xyz=0 -0.230 -0.1 rpy=0 0 1.57

File: urdf/old_model.urdf (robot description, URDF)
Before this commit: robot my_robot, 6 links, 5 joints
Joints:
- joint base_to_left_wheel: axis (none) -> -1 0 0; origin xyz=0 -0.230 -0.1 rpy=0 0 1.57 -> xyz=0 0.230 -0.1 rpy=0 0 1.57
- joint base_to_right_wheel: axis (none) -> 1 0 0; origin xyz=0 0.230 -0.1 rpy=0 0 1.57 -> xyz=0 -0.230 -0.1 rpy=0 0 1.57

Commit message: slam working

File: urdf/my_robot.urdf (robot description, URDF)
Before this commit: robot my_robot, 7 links, 6 joints
Links:
- link lidar: geometry visual cylinder length=0.05 radius=0.1
